File: doc/Kicad/ArduiBodet.kicad_pcb (KiCad board)
At the start: 2 copper layers, 69.8 x 52.6 mm, 22 parts, among them CON1 BARREL_JACK, IC1 ATMEGA328-P, IC2 SN754410, P1 ISP10PIN, P2 DS3231_Breakout_Connector, P3 Moteur Horloge, SW1 SWITCH_INV, SW2 Switch_DPST, U1 LM7805CT

Commit message: Version 1.1. Typon amélioré (pads condos plus larges, espacements,...
Parts:
- C1, C2, C5: footprint Capacitors_ThroughHole:C_Rect_L4_W2.5_P2.5 -> MyLib:C_Rect_L7_W2.5_P2.5
- P1: value ISP10PIN -> ICSP_10_PIN
- P2: footprint Pin_Headers:Pin_Header_Straight_1x05 -> Pin_Headers:Pin_Header_Straight_1x06
- moved C1 41.5 mm to (143.5, 92.7), turned to 0 degrees
- moved C2 38.6 mm to (163.8, 125.5), turned to 180 degrees
- moved R2 6.61 mm to (170.2, 130.8)
- moved IC2 6.35 mm to (154.9, 132.1)
- moved P3 2.90 mm to (178.1, 128.3)
- moved C5 2.54 mm to (175.3, 92.7)
Routing:
- net GNDA: track 285.6 -> 294.8 mm
- net Net-(C1-Pad1): track 157.6 -> 166.1 mm
- net Net-(IC2-Pad3): track 44.0 -> 50.4 mm
- net Net-(IC1-Pad15): track 30.1 -> 36.3 mm
- net Net-(IC1-Pad16): track 40.6 -> 46.8 mm
- net Net-(C4-Pad1): track 167.6 -> 172.7 mm
- net Net-(P3-Pad1): track 4.57 -> 7.93 mm
Other:
- board text added: "ArduiBodet V1.1 (c) Patrice Godard"
- board text removed: "ArduiBodet V1.0 (c) Patrice Godard"
